File: crossover_v1.kicad_sch (KiCad schematic)
At the start: 17 parts, among them J1 POWER, J2 IN, J3 OUT, J4 OUT, J5 OUT, U1 TL082

Commit message: agregando control de volumen de medios, corrigiendo espacio de potenciometro doble
Parts:
- removed H3: MountingHole, MountingHole:MountingHole_3.2mm_M3_DIN965_Pad, symbol Mechanical:MountingHole
- added RV4: 5K, Potentiometer_THT:Potentiometer_Alps_RK163_Dual_Horizontal, symbol Device:R_Potentiometer_Dual
- RV3: footprint Potentiometer_THT:Potentiometer_Piher_T-16H_Double_Horizontal -> Potentiometer_THT:Potentiometer_Alps_RK163_Dual_Horizontal
Connections:
- net DERECHO: now also RV4.5
- net GND: now also J4.2 (Pin_2), RV4.1, RV4.4; no longer J4.3 (Pin_3)
- net IZQUIERDO: now also J4.3 (Pin_3), RV4.2; no longer J4.2 (Pin_2)
- new net filtroPasaAltas/OUT: RV4.3
- new net filtroPasaAltas1/OUT: RV4.6
Other:
- moved on the sheet: J4

Commit message: agregando archivos pdf
Other:
- company: (none) -> Maykol Rey
- title: (none) -> Crossover
- moved on the sheet: J4, RV3, RV4
