File: pasa-bajo-ajust.kicad_sch (KiCad schematic)
At the start: 8 parts, among them U1 TL082

Commit message: agregando control de volumen de medios, corrigiendo espacio de potenciometro doble
Parts:
- RV2: footprint Potentiometer_THT:Potentiometer_Piher_T-16H_Double_Horizontal -> Potentiometer_THT:Potentiometer_Alps_RK163_Dual_Horizontal
Changed lines of the file:
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@@
     (property "Reference" "RV2" (id 0) (at 130.81 104.9782 0))
     (property "Value" "100K" (id 1) (at 130.81 107.2896 0))
-    (property "Footprint" "Potentiometer_THT:Potentiometer_Piher_T-16H_Double_Horizontal" (id 2) (at 137.16 100.965 0)
+    (property "Footprint" "Potentiometer_THT:Potentiometer_Alps_RK163_Dual_Horizontal" (id 2) (at 137.16 100.965 0)
       (effects (font (size 1.27 1.27)) hide)
     )

Commit message: agregando archivos pdf
Other:
- company: https://maykolrey.com -> Maykol Rey
- title: Filtro pasa bajos Ajustable 30Hz a 338Hz -> Crossover
